File: FFCs/HelioMax.kicad_sch (KiCad schematic)
At the start: 71 parts, among them J1 Conn_01x01_Pin, J10 Conn_01x07, J11 Conn_01x07, J12 Conn_Telorum_Belt, J13 Conn_to_Telorum_Belt, J4 Conn_C_to_Praetor_Enclave, J5 Conn_R_to_Praetor_Enclave, J6 Conn_01x07, J7 Conn_01x07, J8 Conn_to_Pollex_Cluster, J9 Conn_Pollex_Cluster, SW0:10 SW0:3, SW0:11 SW0:2, SW0:12 SW0:1, SW0:7 SW0:6, SW0:8 SW0:5, SW0:9 SW0:4, SW1:10 SW1:3, SW1:11 SW1:2, SW1:12 SW1:1, SW1:13 SW1:0, SW1:9 SW1:4, SW2:10 SW2:3, SW2:11 SW2:2, SW2:12 SW2:1, SW2:13 SW2:0, SW2:7 SW2:6, SW2:8 SW2:5, SW2:9 SW2:4, SW3:10 SW3:3, SW3:11 SW3:2, SW3:12 SW3:1, SW3:13 SW3:0, SW3:8 SW3:5, SW3:9 SW3:4, SW4:10 SW4:3, SW4:11 SW4:2, SW4:12 SW4:1, SW4:13 SW4:0, SW4:7 SW4:6, SW4:8 SW4:5, SW4:9 SW4:4, SW5:10 SW5:3, SW5:11 SW5:2, SW5:12 SW5:1, SW5:13 SW5:0, SW5:7 SW5:6, SW5:8 SW5:5, SW5:9 SW5:4, SW6:10 SW6:3, SW6:11 SW6:2, SW6:12 SW6:1, SW6:13 SW6:0, SW6:7 SW6:6, SW6:8 SW6:5, SW6:9 SW6:4

Commit message: added caps and ground planes. Fixed stuff.
Parts:
- added C1: C_Polarized, Capacitor_THT:CP_Radial_D4.0mm_P2.00mm, symbol Device:C_Polarized
- added C2: C, Capacitor_THT:C_Rect_L7.0mm_W2.5mm_P5.00mm, symbol Device:C
Connections:
- net COL0: now also A1.10 (GPIO7), A1.27 (GPIO21), J11.1 (Pin_1), J7.1 (Pin_1)
- net COL1: now also A1.11 (GPIO8), A1.29 (GPIO22), J11.2 (Pin_2), J7.2 (Pin_2)
- net COL2: now also A1.12 (GPIO9), A1.TP4 (~{SMPS_PS}), J11.3 (Pin_3), J7.3 (Pin_3)
- net COL3: now also A1.14 (GPIO10), J1.1 (Pin_1), J11.4 (Pin_4), J7.5 (Pin_5)
- net COL4: now also A1.15 (GPIO11), A1.TP5 (LED_OUT), J11.5 (Pin_5), J7.6 (Pin_6)
- net COL5: now also A1.16 (GPIO12), A1.31 (GPIO26_ADC0), J11.6 (Pin_6), J7.7 (Pin_7)
- net COL6: now also A1.17 (GPIO13), A1.32 (GPIO27_ADC1), J11.8 (Pin_8), J7.8 (Pin_8)
- net GND: now also J10.3 (Pin_3), J11.7 (Pin_7), J6.6 (Pin_6), J7.4 (Pin_4), C1.2, C2.2
- net ROW0: now also A1.1 (GPIO0), A1.19 (GPIO14), J10.1 (Pin_1), J6.1 (Pin_1)
- net ROW1: now also A1.2 (GPIO1), A1.20 (GPIO15), J10.2 (Pin_2), J6.2 (Pin_2)
- net ROW2: now also A1.21 (GPIO16), A1.4 (GPIO2), J10.4 (Pin_4), J6.3 (Pin_3)
- net ROW3: now also A1.22 (GPIO17), A1.5 (GPIO3), J10.5 (Pin_5), J6.4 (Pin_4)
- net ROW4: now also A1.24 (GPIO18), A1.6 (GPIO4), J10.6 (Pin_6), J6.5 (Pin_5)
- net ROW5: now also A1.25 (GPIO19), A1.7 (GPIO5), J10.7 (Pin_7), J6.7 (Pin_7)
- net ROW6: now also A1.26 (GPIO20), A1.9 (GPIO6), J10.8 (Pin_8), J6.8 (Pin_8)
- net at A1.36 (3V3): now also C2.1
- net at A1.40 (VBUS): now also C1.1

Commit message: Fixed FFC connector, grounded the MPs.
Connections:
- net COL1: now also J8.8 (Pin_8), J9.2 (Pin_2); no longer J8.2 (Pin_2), J9.8 (Pin_8)
- net COL2: now also J8.7 (Pin_7), J9.3 (Pin_3); no longer J8.3 (Pin_3), J9.7 (Pin_7)
- net COL3: now also J8.6 (Pin_6), J9.4 (Pin_4); no longer J8.4 (Pin_4), J9.6 (Pin_6)
- net COL5: now also J8.4 (Pin_4), J9.6 (Pin_6); no longer J8.6 (Pin_6), J9.4 (Pin_4)
- net COL6: now also J8.3 (Pin_3), J9.7 (Pin_7); no longer J8.7 (Pin_7), J9.3 (Pin_3)
- net ROW0: now also J8.2 (Pin_2), J9.8 (Pin_8); no longer J8.8 (Pin_8), J9.2 (Pin_2)
Changed lines of the file:
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@@
 		(lib_id "Connector_Generic:Conn_01x09")
 		(at 184.15 167.64 0)
-		(mirror x)
 		(unit 1)
 		(body_style 1)
@@
 		(dnp no)
 		(property "Reference" "J8"
-			(at 186.69 168.9101 0)
+			(at 186.69 166.3699 0)
 			(show_name no)
 			(do_not_autoplace no)
@@
 		)
 		(property "Value" "Conn_to_Pollex_Cluster"
-			(at 186.69 166.3701 0)
+			(at 186.69 168.9099 0)
 			(show_name no)
 			(do_not_autoplace no)
@@
 		(lib_id "Connector_Generic:Conn_01x09")
 		(at 168.91 226.06 0)
+		(mirror x)
 		(unit 1)
 		(body_style 1)
@@
 		(in_pos_files yes)
 		(dnp no)
-		(fields_autoplaced yes)
 		(property "Reference" "J9"
-			(at 171.45 224.7899 0)
+			(at 171.45 227.3301 0)
 			(show_name no)
 			(do_not_autoplace no)
@@
 		)
 		(property "Value" "Conn_Pollex_Cluster"
-			(at 171.45 227.3299 0)
-			(show_name no)
-			(do_not_autoplace no)
+			(at 171.45 224.7901 0)
+			(show_name no)
+			(do_not_autoplace no)
